File: ROCKETRY Camera PCB.kicad_pcb (KiCad board)
At the start: 2 copper layers, 111.8 x 72.9 mm, 38 parts, among them J1 Conn_01x03_Pin, J2 Conn_01x01_Pin, J3 Conn_01x01_Pin, J4 Conn_01x01_Pin, Q1 IRF7780M, U1 3.4v, U2 3.4v, U4 AP62200WU

Commit message: First commit after import to UVR
Other:
- board size 111.8 x 72.9 mm -> 111.8 x 75.7 mm
Changed lines of the file:
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@@
 	(gr_line
 		(start 83.8 74.9)
-		(end 83.82 123.19)
+		(end 83.82 125.984)
 		(stroke
 			(width 0.05)
@@
 			(type default)
 		)
-		(layer "Edge.Cuts")
-	)
-	(gr_circle
-		(center 152.246 110.336)
-		(end 154.151 110.336)
-		(stroke
-			(width 0.05)
-			(type default)
-		)
-		(fill none)
 		(layer "Edge.Cuts")
 	)
@@
 	)
 	(gr_line
-		(start 195.58 123.19)
+		(start 195.58 125.984)
 		(end 195.6 74.9)
 		(stroke
@@
 		(layer "Edge.Cuts")
 	)
-	(gr_circle
-		(center 126.746 110.336)
-		(end 128.651 110.336)
-		(stroke
-			(width 0.05)
-			(type default)
-		)
-		(fill none)
-		(layer "Edge.Cuts")
-	)
 	(gr_line
 		(start 113.03 66.421)
@@
 		(layer "Edge.Cuts")
 	)
-	(gr_circle
-		(center 126.746 84.836)
-		(end 128.651 84.836)
-		(stroke
-			(width 0.05)
-			(type default)
-		)
-		(fill none)
-		(layer "Edge.Cuts")
-	)
 	(gr_line
 		(start 113.03 70.8914)
@@
 		(layer "Edge.Cuts")
 	)
-	(gr_circle
-		(center 152.246 84.836)
-		(end 154.151 84.836)
-		(stroke
-			(width 0.05)
-			(type default)
-		)
-		(fill none)
-		(layer "Edge.Cuts")
-	)
 	(gr_line
 		(start 129.921 120.65)
@@
 	)
 	(gr_line
-		(start 195.58 123.19)
-		(end 83.82 123.19)
-		(stroke
-			(width 0.05)
+		(start 195.58 125.984)
+		(end 83.82 125.984)
+		(stroke
+			(width 0.05)
