File: ROCKETRY Camera PCB.kicad_sch (KiCad schematic)
At the start: 28 parts, among them J1 Conn_01x03_Pin, J2 Conn_01x01_Pin, J3 Conn_01x01_Pin, J4 Conn_01x01_Pin, U3 AP62200WU

Commit message: pcb ready for final review/ ordering
Connections:
- net GND: now also BT2.2 (-), C4.2, D1.1 (K), D3.1 (K), U3.3 (GND)
Changed lines of the file:
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@@
 	(title_block
 		(title "UVR Anduril 2 Camera PCB")
-		(date "Dec 30 2024")
-		(rev "Rev 2")
+		(date "2025-02-11")
+		(rev "Rev 2.1")
 		(company "By: Khephren Gould")
 	)
 	(junction
+		(at 187.96 60.96)
+		(diameter 0)
+		(color 0 0 0 0)
+	)
+	(junction
 		(at 172.72 106.68)
 		(diameter 0)
@@
 	)
 	(junction
+		(at 211.455 50.8)
+		(diameter 0)
+		(color 0 0 0 0)
+	)
+	(junction
 		(at 173.7281 111.76)
 		(diameter 0)
@@
 	)
 	(junction
+		(at 124.46 58.42)
+		(diameter 0)
+		(color 0 0 0 0)
+	)
+	(junction
 		(at 88.2142 111.0996)
 		(diameter 0)
@@
 	)
 	(junction
+		(at 89.535 66.04)
+		(diameter 0)
+		(color 0 0 0 0)
+	)
+	(junction
 		(at 211.455 35.56)
 		(diameter 0)
@@
 	)
 	(junction
+		(at 172.72 58.42)
+		(diameter 0)
+		(color 0 0 0 0)
+	)
+	(junction
+		(at 198.12 60.96)
+		(diameter 0)
+		(color 0 0 0 0)
+	)
+	(junction
 		(at 165.1 39.3657)
 		(diameter 0)
@@
 	(wire
 		(pts
+			(xy 89.535 66.04) (xy 107.95 66.04)
+		)
+		(stroke
+			(width 0)
+			(type default)
+		)
+	)
+	(wire
+		(pts
 			(xy 217.17 134.62) (xy 222.25 134.62)
 		)
@@
 	(wire
 		(pts
-			(xy 172.72 55.88) (xy 172.72 60.96)
+			(xy 172.72 55.88) (xy 172.72 58.42)
 		)
 		(stroke
@@
 	(wire
 		(pts
+			(xy 175.26 58.42) (xy 172.72 58.42)
+		)
+		(stroke
+			(width 0)
+			(type default)
+		)
+	)
+	(wire
+		(pts
 			(xy 98.3742 108.5596) (xy 98.3742 111.0996)
 		)
@@
 	(wire
 		(pts
+			(xy 198.12 60.96) (xy 198.12 63.5)
+		)
+		(stroke
+			(width 0)
+			(type default)
+		)
+	)
+	(wire
+		(pts
 			(xy 204.47 147.32) (xy 204.47 149.86)
 		)
@@
 	(wire
 		(pts
-			(xy 187.96 49.53) (xy 187.96 63.5)
+			(xy 187.96 49.53) (xy 187.96 60.96)
 		)
 		(stroke
@@
 	(wire
 		(pts
-			(xy 198.12 49.53) (xy 198.12 63.5)
+			(xy 198.12 49.53) (xy 198.12 60.96)
 		)
 		(stroke
@@
 	(wire
 		(pts
+			(xy 124.46 58.42) (xy 107.95 58.42)
+		)
+		(stroke
+			(width 0)
+			(type default)
+		)
+	)
+	(wire
+		(pts
+			(xy 211.455 50.8) (xy 205.74 50.8)
+		)
+		(stroke
+			(width 0)
+			(type default)
+		)
+	)
+	(wire
+		(pts
+			(xy 205.74 60.96) (xy 198.12 60.96)
+		)
+		(stroke
+			(width 0)
+			(type default)
+		)
+	)
+	(wire
+		(pts
 			(xy 201.93 87.9576) (xy 201.93 96.52)
 		)
@@
 	(wire
 		(pts
+			(xy 175.26 60.96) (xy 175.26 58.42)
+		)
+		(stroke
+			(width 0)
+			(type default)
+		)
+	)
+	(wire
+		(pts
 			(xy 172.72 106.68) (xy 191.77 106.68)
 		)
@@
 	(wire
 		(pts
+			(xy 187.96 60.96) (xy 187.96 63.5)
+		)
+		(stroke
+			(width 0)
+			(type default)
+		)
+	)
+	(wire
+		(pts
+			(xy 187.96 60.96) (xy 175.26 60.96)
+		)
+		(stroke
+			(width 0)
+			(type default)
+		)
+	)
+	(wire
+		(pts
+			(xy 187.96 60.96) (xy 198.12 60.96)
+		)
+		(stroke
+			(width 0)
+			(type default)
+		)
+	)
+	(wire
+		(pts
 			(xy 19.05 44.0508) (xy 28.702 44.0508)
 		)
@@
 	(wire
 		(pts
+			(xy 205.74 50.8) (xy 205.74 60.96)
+		)
+		(stroke
+			(width 0)
+			(type default)
+		)
+	)
+	(wire
+		(pts
 			(xy 172.72 35.56) (xy 181.61 35.56)
 		)
@@
 	(wire
 		(pts
+			(xy 107.95 58.42) (xy 107.95 66.04)
+		)
+		(stroke
+			(width 0)
+			(type default)
+		)
+	)
+	(wire
+		(pts
 			(xy 207.01 147.32) (xy 207.01 149.86)
 		)
@@
 	(wire
 		(pts
+			(xy 124.46 58.42) (xy 172.72 58.42)
+		)
+		(stroke
+			(width 0)
+			(type default)
+		)
+	)
+	(wire
+		(pts
 			(xy 211.455 35.56) (xy 226.06 35.56)
 		)
@@
 		)
 		(stroke
+			(width 0)
+			(type default)
+		)
+	)
+	(wire
+		(pts
+			(xy 172.72 58.42) (xy 172.72 60.96)
+		)
+		(stroke

Commit message: adding curves to pcb edges
Parts:
- added J5: Conn_01x02_Pin, symbol Connector:Conn_01x02_Pin
Connections:
- net VCC: now also J5.2 (Pin_2); no longer C4.1, R8.1, U3.1 (VIN)
- new net: C4.1, J5.1 (Pin_1), R8.1, U3.1 (VIN)
Changed lines of the file:
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@@
+	(wire
+		(pts
+			(xy 59.69 38.1) (xy 59.69 41.9608)
+		)
+		(stroke
+			(width 0)
+			(type default)
+		)
+	)
 	(wire
 		(pts
@@
 	(wire
 		(pts
+			(xy 62.23 41.9608) (xy 73.6092 41.9608)
+		)
+		(stroke
+			(width 0)
+			(type default)
+		)
+	)
+	(wire
+		(pts
 			(xy 177.165 109.22) (xy 191.77 109.22)
 		)
@@
 	(wire
 		(pts
-			(xy 44.5262 41.9608) (xy 73.6092 41.9608)
-		)
-		(stroke
-			(width 0)
-			(type default)
-		)
-	)
-	(wire
-		(pts
 			(xy 28.6677 35.3992) (xy 33.7541 35.3992)
 		)
@@
 	(wire
 		(pts
+			(xy 62.23 38.1) (xy 62.23 41.9608)
+		)
+		(stroke
+			(width 0)
+			(type default)
+		)
+	)
+	(wire
+		(pts
 			(xy 44.4754 41.91) (xy 44.5262 41.9608)
 		)
@@
 		(pts
 			(xy 73.66 41.91) (xy 89.535 41.91)
+		)
+		(stroke
+			(width 0)
+			(type default)
+		)
+	)
+	(wire
+		(pts
+			(xy 59.69 41.9608) (xy 44.5262 41.9608)
 		)
 		(stroke
@@
 					(unit 1)
 				)
+			)
+		)
+	)
+	(symbol
+		(lib_id "Connector:Conn_01x02_Pin")
+		(at 62.23 33.02 270)
+		(unit 1)
+		(exclude_from_sim no)
+		(in_bom yes)
+		(on_board yes)
+		(dnp no)
+		(fields_autoplaced yes)
+		(property "Reference" "J5"
+			(at 63.5 32.3849 90)
+			(effects
+				(font
+					(size 1.27 1.27)
+				)
+				(justify left)
+			)
+		)
+		(property "Value" "Conn_01x02_Pin"
+			(at 63.5 34.9249 90)
+			(effects
+				(font
+					(size 1.27 1.27)
+				)
+				(justify left)
+			)
+		)
+		(property "Footprint" ""
+			(at 62.23 33.02 0)
+			(effects
+				(font
+					(size 1.27 1.27)
+				)
+				(hide yes)
+			)
+		)
+		(property "Datasheet" "~"
+			(at 62.23 33.02 0)
+			(effects
+				(font
+					(size 1.27 1.27)
+				)
+				(hide yes)
+			)
+		)
+		(property "Description" "Generic connector, single row, 01x02, script generated"
+			(at 62.23 33.02 0)
+			(effects
+				(font
+					(size 1.27 1.27)
+				)
+				(hide yes)
+			)
+		)
+		(pin "1"
+		)
+		(pin "2"
+		)
+		(instances
+			(project ""
+				(path "/977e3c33-6744-4a35-9b77-0633aa2ba496"
+					(reference "J5")
+					(unit 1)
+				)

Commit message: added curves to pcb edges, added connector for screw switch
Parts:
- J1: footprint Connector_Molex:Molex_PicoBlade_53047-0310_1x03_P1.25mm_Vertical -> Connector_JST:JST_XH_B4B-XH-A_1x04_P2.50mm_Vertical
- J5: footprint (none) -> Connector_JST:JST_XH_B2B-XH-A_1x02_P2.50mm_Vertical
Changed lines of the file:
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@@
 	(title_block
 		(title "UVR Anduril 2 Camera PCB")
-		(date "2025-02-11")
-		(rev "Rev 2.1")
+		(date "2025-02-15")
+		(rev "Rev 2.2")
 		(company "By: Khephren Gould")
 	)
@@
 			)
 		)
-		(property "Footprint" ""
+		(property "Footprint" "Connector_JST:JST_XH_B2B-XH-A_1x02_P2.50mm_Vertical"
 			(at 62.23 33.02 0)
 			(effects
@@
 		)
 		(instances
-			(project ""
+			(project "ROCKETRY Camera PCB"
 				(path "/977e3c33-6744-4a35-9b77-0633aa2ba496"
 					(reference "J5")
@@
 			)
 		)
-		(property "Footprint" "Connector_Molex:Molex_PicoBlade_53047-0310_1x03_P1.25mm_Vertical"
+		(property "Footprint" "Connector_JST:JST_XH_B4B-XH-A_1x04_P2.50mm_Vertical"
 			(at 158.75 109.22 0)
 			(effects

Commit message: made critical updates based on Aila's feedback
Parts:
- removed J2, J3: Conn_01x01_Pin, Connector_PinHeader_1.00mm:PinHeader_1x01_P1.00mm_Vertical, symbol Connector:Conn_01x01_Pin
- added J4: Conn_01x01_Pin, Connector_PinHeader_1.00mm:PinHeader_1x01_P1.00mm_Vertical, symbol Connector:Conn_01x01_Pin
- added R5: 0, Resistor_SMD:R_0402_1005Metric_Pad0.72x0.64mm_HandSolder, symbol Device:R_US
- added R8: 10k, Resistor_SMD:R_0603_1608Metric_Pad0.98x0.95mm_HandSolder, symbol Device:R_US
- renumbered C2 to C1, C4 to C2, C5 to C3, C6 to C4, C7 to C5, C8 to C6, C9 to C7, C10 to C8, J5 to J1, J1 to J2, J4 to J5, R8 to R1, R9 to R2, R10 to R3, R11 to R4, R12 to R7, U2 to U1, U3 to U2
Connections:
- net +5V: now also R5.1, R8.1; no longer C5.1, J2.3 (Pin_3), R4.1
- net GND: now also U1.2 (I2), U1.3 (SNO), U1.4 (CS), U1.9 (INT)
- net at A1.27 (+5V): now also J4.1 (Pin_1)
- net at A1.28 (~{RESET}): now also A1.3 (~{RESET}), R8.2
- new net: C5.1, J2.3 (Pin_3), R4.1, R5.2
- no-connect marks 29 -> 22

Commit message: finished with updates, has my approval to order
Parts:
- J4: footprint Connector_PinHeader_1.00mm:PinHeader_1x01_P1.00mm_Vertical -> custom:mouonting_hole
Connections:
- net GND: now also A1.10 (D7), A1.11 (D8), A1.12 (D9), A1.13 (D10), A1.14 (D11), A1.15 (D12), A1.16 (D13), A1.18 (AREF), A1.19 (A0), A1.20 (A1), A1.21 (A2), A1.22 (A3), A1.25 (A6), A1.26 (A7), A1.5 (D2), A1.6 (D3), A1.7 (D4), A1.8 (D5), A1.9 (D6)
- no-connect marks 22 -> 3
