File: _autosave-ROCKETRY Camera PCB.kicad_sch (KiCad schematic)
At the start: 30 parts, among them J1 Conn_01x02_Pin, J2 Conn_01x03_Pin, J4 Conn_01x01_Pin, J5 Conn_01x01_Pin, U2 AP62200WU

Commit message: exported gerbers
Connections:
- net GND: now also U2.1 (GND); no longer U2.3 (GND)
- net at C4.2, R2.2, R3.1: now also U2.4 (FB); no longer U2.6 (FB)
- net at C2.1, J1.1 (Pin_1), R1.1: now also U2.3 (VIN); no longer U2.1 (VIN)
- net at C3.2: now also U2.6 (BST); no longer U2.4 (BST)
